Commit message: fourth

File: gp/urdf/caster_wheel.xacro (robot description, xacro)
@@ -3,4 +3,9 @@
     <!-- Caster Wheel Link -->
     <link name="caster_wheel_link">
+      <visual>
+        <geometry>
+          <sphere radius="${caster_wheel_radius}"/>
+        </geometry>
+      </visual>
       <collision>
         <geometry>
@@ -12,4 +17,38 @@
       </xacro:inertial_sphere>
     </link>
+    <link name="caster2_wheel_link">
+      <visual>
+        <geometry>
+          <sphere radius="${caster_wheel_radius}"/>
+        </geometry>
+      </visual>
+      <collision>
+        <geometry>
+          <sphere radius="${caster_wheel_radius}"/>
+        </geometry>
+      </collision>
+      <xacro:inertial_sphere mass="${caster_wheel_mass}" radius="${caster_wheel_radius}">
+        <origin xyz="0.0 0.0 0.0" rpy="0.0 0.0 0.0"/>
+      </xacro:inertial_sphere>
+    </link>
+    <joint name="caster_wheel2_joint" type="fixed">
+      <origin xyz="${-caster_wheel_offset_x} 0.0 ${caster_wheel_offset_z}" rpy="0.0 0.0 0.0"/>
+      <parent link="chassis_link"/>
+      <child link="caster2_wheel_link"/>
+    </joint>
+    <link name="caster2_holder">
+      <visual>
+        <geometry>
+          <cylinder radius="${caster_wheel_radius/2}" length="${caster_wheel_offset_z*2}"/>
+        </geometry>
+        <material name="blue"/>
+      </visual>
+    </link>
+    <!-- Holder Joint -->
+    <joint name="holder2_joint" type="fixed">
+      <origin xyz="${-caster_wheel_offset_x} 0.0 0.0" rpy="0.0 0.0 0.0"/>
+      <parent link="chassis_link"/>
+      <child link="caster2_holder"/>
+    </joint>
     <!-- Caster Wheel Joint -->
     <joint name="caster_wheel_joint" type="fixed">

File: gp/urdf/chassis.xacro (robot description, xacro)
@@ -7,5 +7,5 @@
                 <cylinder radius="0.25" length="0.1"/>
             </geometry>
-            <origin xyz="0 0 0.3" rpy="0 0 0"/>
+            <origin xyz="0 0 0.095" rpy="0 0 0"/>
         </visual>
         <collision>
@@ -13,8 +13,8 @@
                 <cylinder radius="0.25" length="0.1"/>
             </geometry>
-            <origin xyz="0 0 0.3" rpy="0 0 0"/>
+            <origin xyz="0 0 0.095" rpy="0 0 0"/>
         </collision>
         <inertial>
-            <origin xyz="0 0 0.3" rpy="0 0 0"/>
+            <origin xyz="0 0 0.095" rpy="0 0 0"/>
             <mass value="9.0"/>
             <inertia
@@ -24,28 +24,4 @@
         </inertial>
     </link>
-    <!-- Wheel Link -->
-    <!-- <link name="wheel_link">
-        <visual>
-            <geometry>
-                <cylinder radius="0.095" length="0.05"/>
-            </geometry>
-            <origin xyz="0.3 0 0.095" rpy="0 1.5708 0"/>
-        </visual>
-        <collision>
-            <geometry>
-                <cylinder radius="0.095" length="0.05"/>
-            </geometry>
-            <origin xyz="0.3 0 0.095" rpy="0 1.5708 0"/>
-        </collision>
-        <inertial>
-            <origin xyz="0.3 0 0.095" rpy="0 1.5708 0"/>
-            <mass value="0.25"/>
-            <inertia
-              ixx="0.000307" ixy="0.0" ixz="0.0"
-              iyy="0.000307" iyz="0.0"
-              izz="0.0001535"/>
-        </inertial>
-    </link> -->
-    <!-- Chassis Joint -->
     <joint name="chassis_joint" type="fixed">
         <parent link="base_link"/>
@@ -53,9 +29,3 @@
         <origin xyz="0 0 0" rpy="0 0 0"/>
     </joint>
-    <!-- Wheel Joint -->
-    <!-- <joint name="wheel_joint" type="continuous">
-        <parent link="chassis_link"/>
-        <child link="wheel_link"/>
-        <origin xyz="0 0 -0.3" rpy="0 0 0"/>
-    </joint> -->
 </robot>

File: gp/urdf/properties.xacro (robot description, xacro)
@@ -3,20 +3,19 @@
     <!-- Properties -->
     <!-- Chassis -->
-    <xacro:property name="chassis_length" value="0.4"/>
-    <xacro:property name="chassis_width" value="0.3"/>
-    <xacro:property name="chassis_height" value="0.11"/>
-    <xacro:property name="chassis_mass" value="2.0"/>
+    <xacro:property name="chassis_radius" value="0.25"/>
+    <xacro:property name="chassis_length" value="0.1"/>
+    <xacro:property name="chassis_mass" value="9.0"/>
     <!-- Wheels -->
-    <xacro:property name="wheel_offset_x" value="0.1285"/>
-    <xacro:property name="wheel_offset_y" value="0.112"/>
-    <xacro:property name="wheel_offset_z" value="-0.025"/>
-    <xacro:property name="wheel_thickness" value="0.027"/>
-    <xacro:property name="wheel_radius" value="0.0325"/>
+    <xacro:property name="wheel_offset_x" value="0.0"/> <!-- Centered on x-axis -->
+    <xacro:property name="wheel_offset_y" value="0.25"/> <!-- Adjusted for the new radius -->
+    <xacro:property name="wheel_offset_z" value="0.05"/> <!-- Adjusted for the new thickness -->
+    <xacro:property name="wheel_thickness" value="0.04"/> <!-- 4 cm -->
+    <xacro:property name="wheel_radius" value="0.095"/> <!-- 9.5 cm -->
     <xacro:property name="wheel_mass" value="0.037"/>
     <!-- Caster Wheel -->
-    <xacro:property name="caster_wheel_radius" value="0.01"/>
-    <xacro:property name="caster_wheel_mass" value="0.01"/>
-    <xacro:property name="caster_wheel_offset_x" value="0.370"/>
-    <xacro:property name="caster_wheel_offset_z" value="0.045"/>
+    <xacro:property name="caster_wheel_radius" value="0.015"/> <!-- Increased size -->
+    <xacro:property name="caster_wheel_mass" value="0.05"/> <!-- Increased mass -->
+    <xacro:property name="caster_wheel_offset_x" value="0.15"/> <!-- Positioned forward -->
+    <xacro:property name="caster_wheel_offset_z" value="-0.045"/>
     <!-- Colors -->
     <material name="white">
@@ -35,3 +34,3 @@
       <color rgba="0 0 0 1"/>
     </material>
-  </robot>
+</robot>

File: gp/urdf/robot.urdf.xacro (robot description, xacro)
@@ -1,7 +1,7 @@
 <?xml version="1.0"?>
 <robot xmlns:xacro="http://www.ros.org/wiki/xacro" name="gp">
+    <xacro:include filename="properties.xacro"/>
     <xacro:include filename="inertial_macros.xacro"/>
     <xacro:include filename="chassis.xacro"/>
-    <xacro:include filename="properties.xacro"/>
     <xacro:include filename="wheels.xacro"/>
     <xacro:include filename="caster_wheel.xacro"/>

File: gp/urdf/wheels.xacro (robot description, xacro)
@@ -1,35 +1,38 @@
-<?xml version="1.0"?>
 <robot xmlns:xacro="http://www.ros.org/wiki/xacro">
-    <!-- Caster Wheel Link -->
-    <link name="caster_wheel_link">
+  <!-- Wheel Link Macro -->
+  <xacro:macro name="wheel_link" params="link_name">
+    <link name="${link_name}">
       <collision>
         <geometry>
-          <sphere radius="${caster_wheel_radius}"/>
+          <cylinder radius="${wheel_radius}" length="${wheel_thickness}"/>
         </geometry>
       </collision>
-      <xacro:inertial_sphere mass="${caster_wheel_mass}" radius="${caster_wheel_radius}">
-        <origin xyz="0.0 0.0 0.0" rpy="0.0 0.0 0.0"/>
-      </xacro:inertial_sphere>
-    </link>
-    <!-- Caster Wheel Joint -->
-    <joint name="caster_wheel_joint" type="fixed">
-      <origin xyz="${caster_wheel_offset_x} 0.0 ${caster_wheel_offset_z}" rpy="0.0 0.0 0.0"/>
-      <parent link="chassis_link"/>
-      <child link="caster_wheel_link"/>
-    </joint>
-    <!-- Caster Holder (Only for visuals) -->
-    <link name="caster_holder">
       <visual>
         <geometry>
-          <cylinder radius="${caster_wheel_radius/2}" length="${caster_wheel_offset_z*2}"/>
+          <cylinder radius="${wheel_radius}" length="${wheel_thickness}"/>
         </geometry>
-        <material name="blue"/>
+        <material name="white"/>
       </visual>
+      <xacro:inertial_cylinder mass="${wheel_mass}" length="${wheel_thickness}" radius="${wheel_radius}">
+        <origin xyz="0 0 0" rpy="0 0 0"/>
+      </xacro:inertial_cylinder>
     </link>
-    <!-- Holder Joint -->
-    <joint name="holder_joint" type="fixed">
-      <origin xyz="${caster_wheel_offset_x} 0.0 0.0" rpy="0.0 0.0 0.0"/>
-      <parent link="chassis_link"/>
-      <child link="caster_holder"/>
+  </xacro:macro>
+  <!-- Wheel Joint Macro -->
+  <xacro:macro name="wheel_joint" params="joint_name wheel_name x_offset y_offset roll">
+    <joint name="${joint_name}" type="continuous">
+      <origin xyz="${x_offset} ${y_offset} ${wheel_offset_z}" rpy="${roll} 0.0 0.0"/>
+      <parent link="base_link"/>
+      <child link="${wheel_name}"/>
+      <axis xyz="0.0 0.0 1"/>
     </joint>
-  </robot>
+  </xacro:macro>
+  <!-- Left Wheel Link -->
+  <xacro:wheel_link link_name="left_wheel_link"/>
+  <!-- Left Wheel Joint -->
+  <xacro:wheel_joint joint_name="left_wheel_joint" wheel_name="left_wheel_link" x_offset="${wheel_offset_x}" y_offset="${wheel_offset_y}" roll="${-pi/2}"/>
+  <!-- Right Wheel Link -->
+  <xacro:wheel_link link_name="right_wheel_link"/>
+  <!-- Right Wheel Joint -->
+  <xacro:wheel_joint joint_name="right_wheel_joint" wheel_name="right_wheel_link" x_offset="${wheel_offset_x}" y_offset="${-wheel_offset_y}" roll="${pi/2}"/>
+</robot>

Commit message: fifth

File: gp/urdf/caster_wheel.xacro (robot description, xacro)
@@ -72,3 +72,11 @@
       <child link="caster_holder"/>
     </joint>
+    <gazebo refernce="caster2_wheel_link">
+      <mu1 value="0.001"/>
+      <mu2 value="0.001"/>
+    </gazebo>
+    <gazebo refernce="caster_wheel_link">
+      <mu1 value="0.001"/>
+      <mu2 value="0.001"/>
+    </gazebo>
   </robot>

File: gp/urdf/chassis.xacro (robot description, xacro)
@@ -29,3 +29,6 @@
         <origin xyz="0 0 0" rpy="0 0 0"/>
     </joint>
+   <gazebo refernce="chassis_link">
+        <material> Gazebo/Grey </material>
+   </gazebo>
 </robot>

File: gp/urdf/properties.xacro (robot description, xacro)
@@ -17,5 +17,5 @@
     <xacro:property name="caster_wheel_mass" value="0.05"/> <!-- Increased mass -->
     <xacro:property name="caster_wheel_offset_x" value="0.15"/> <!-- Positioned forward -->
-    <xacro:property name="caster_wheel_offset_z" value="-0.045"/>
+    <xacro:property name="caster_wheel_offset_z" value="-0.025"/>
     <!-- Colors -->
     <material name="white">

File: gp/urdf/robot.urdf.xacro (robot description, xacro)
@@ -6,4 +6,5 @@
     <xacro:include filename="wheels.xacro"/>
     <xacro:include filename="caster_wheel.xacro"/>
+    <xacro:include filename="gazebo_control.xacro"/>
     <link name="base_link"/>
 </robot>

File: gp/urdf/wheels.xacro (robot description, xacro)
@@ -20,7 +20,7 @@
   </xacro:macro>
   <!-- Wheel Joint Macro -->
-  <xacro:macro name="wheel_joint" params="joint_name wheel_name x_offset y_offset roll">
+  <xacro:macro name="wheel_joint" params="joint_name wheel_name x_offset y_offset ">
     <joint name="${joint_name}" type="continuous">
-      <origin xyz="${x_offset} ${y_offset} ${wheel_offset_z}" rpy="${roll} 0.0 0.0"/>
+      <origin xyz="${x_offset} ${y_offset} ${wheel_offset_z}" rpy="${-pi/2} 0.0 0.0"/>
       <parent link="base_link"/>
       <child link="${wheel_name}"/>
@@ -31,8 +31,14 @@
   <xacro:wheel_link link_name="left_wheel_link"/>
   <!-- Left Wheel Joint -->
-  <xacro:wheel_joint joint_name="left_wheel_joint" wheel_name="left_wheel_link" x_offset="${wheel_offset_x}" y_offset="${wheel_offset_y}" roll="${-pi/2}"/>
+  <xacro:wheel_joint joint_name="left_wheel_joint" wheel_name="left_wheel_link" x_offset="${wheel_offset_x}" y_offset="${wheel_offset_y}" />
   <!-- Right Wheel Link -->
   <xacro:wheel_link link_name="right_wheel_link"/>
   <!-- Right Wheel Joint -->
-  <xacro:wheel_joint joint_name="right_wheel_joint" wheel_name="right_wheel_link" x_offset="${wheel_offset_x}" y_offset="${-wheel_offset_y}" roll="${pi/2}"/>
+  <xacro:wheel_joint joint_name="right_wheel_joint" wheel_name="right_wheel_link" x_offset="${wheel_offset_x}" y_offset="${-wheel_offset_y}" />
+  <gazebo refernce="left_wheel_link">
+    <material> Gazebo/Black </material>
+</gazebo>
+<gazebo refernce="right_wheel_link">
+  <material> Gazebo/Black </material>
+</gazebo>
 </robot>
