Commit message: nav

File: gp/urdf/robot.urdf.xacro (robot description, xacro)
@@ -10,3 +10,8 @@
     <xacro:include filename="lidar.xacro"/>
     <link name="base_link"/>
+    <link name="base_footprint"/>
+    <joint name="base_footprint_joint" type="fixed">
+        <parent link="base_link"/>
+        <child link="base_footprint"/>
+    </joint>
 </robot>
